File: ImpactInsole_v1/ImpactInsole_v1.kicad_pcb (KiCad board)
At the start: 2 copper layers, 5 parts, among them J1 503480-1800, J2 Conn_01x02, U1 CD74HC4067SM96, U2 ADC081S021CIMF, U3 LD1117S33TR_SOT223

Commit message: pcb begnnings + more libs
Parts:
- added C1: 0.1u, Capacitor_SMD:C_0603_1608Metric_Pad1.08x0.95mm_HandSolder, B.Cu at (150.8, 59.8)
- added C10: 1u, Capacitor_SMD:C_0603_1608Metric_Pad1.08x0.95mm_HandSolder, F.Cu at (142.0, 59.8)
- added C2: 100n, Capacitor_SMD:C_0603_1608Metric_Pad1.08x0.95mm_HandSolder, B.Cu at (144.2, 61.7)
- added C3: 100n, Capacitor_SMD:C_0603_1608Metric_Pad1.08x0.95mm_HandSolder, F.Cu at (141.2, 64.0)
- added C4: 0.1u, Capacitor_SMD:C_0603_1608Metric_Pad1.08x0.95mm_HandSolder, F.Cu at (157.6, 72.2)
- added C5: 1u, Capacitor_SMD:C_0603_1608Metric_Pad1.08x0.95mm_HandSolder, F.Cu at (160.3, 68.6)
- added C6: 10u, Capacitor_SMD:C_0603_1608Metric_Pad1.08x0.95mm_HandSolder, F.Cu at (137.8, 54.1)
- added C7: 10n, Capacitor_SMD:C_0603_1608Metric_Pad1.08x0.95mm_HandSolder, F.Cu at (135.3, 53.9)
- added C8: 0.1u, Capacitor_SMD:C_0603_1608Metric_Pad1.08x0.95mm_HandSolder, F.Cu at (148.2, 84.2)
- added C9: 10u, Capacitor_SMD:C_0603_1608Metric_Pad1.08x0.95mm_HandSolder, F.Cu at (145.6, 56.8)
- added J3: USB_C_Receptacle_USB2.0_16P, Connector_USB:USB_C_Receptacle_G-Switch_GT-USB-7010ASV, F.Cu at (121.3, 61.9)
- added R1: 4.7k, Resistor_SMD:R_0603_1608Metric_Pad0.98x0.95mm_HandSolder, F.Cu at (148.4, 64.8)
- added R10: 10k, Resistor_SMD:R_0603_1608Metric_Pad0.98x0.95mm_HandSolder, F.Cu at (138.4, 62.0)
- added R2: 4.7k, Resistor_SMD:R_0603_1608Metric_Pad0.98x0.95mm_HandSolder, F.Cu at (142.5, 66.6)
- added R3: 5.1k, Resistor_SMD:R_0603_1608Metric_Pad0.98x0.95mm_HandSolder, B.Cu at (126.6, 59.2)
- added R4: 5.1k, Resistor_SMD:R_0603_1608Metric_Pad0.98x0.95mm_HandSolder, B.Cu at (126.7, 62.7)
- added R5: 30k, Resistor_SMD:R_0603_1608Metric_Pad0.98x0.95mm_HandSolder, F.Cu at (160.0, 62.9)
- added R6: 4.7k, Resistor_SMD:R_0603_1608Metric_Pad0.98x0.95mm_HandSolder, F.Cu at (160.4, 66.6)
- added R7: 10k, Resistor_SMD:R_0603_1608Metric_Pad0.98x0.95mm_HandSolder, F.Cu at (129.6, 57.3)
- added R8: 2.2k, Resistor_SMD:R_0603_1608Metric_Pad0.98x0.95mm_HandSolder, B.Cu at (137.7, 57.0)
- added R9: 4k, Resistor_SMD:R_0603_1608Metric_Pad0.98x0.95mm_HandSolder, F.Cu at (132.7, 54.9)
- added TP1: TestPoint, TestPoint:TestPoint_THTPad_1.0x1.0mm_Drill0.5mm, F.Cu at (135.2, 63.1)
- added U4: LSM6DSOXTR, IMU_Senior_Design:PQFN50P250X300X86-14N, F.Cu at (144.3, 63.8)
- added U5: BQ24075RGTR, pp_senior_design:QFN50P300X300X100-17N, F.Cu at (135.0, 58.1)
- added U6: ESP32-S3-WROOM-1, RF_Module:ESP32-S3-WROOM-1, F.Cu at (137.2, 81.1)
- added U7: MCP1700x-300xxTT, Package_TO_SOT_SMD:SOT-23, F.Cu at (142.2, 55.9)
- J2: footprint Connector_JST:JST_PH_B2B-PH-K_1x02_P2.00mm_Vertical -> conn_sen:JST_S2B-PH-K-S_LF__SN_
- U3: value LD1117S33TR_SOT223 -> OPA1662D; footprint Package_TO_SOT_SMD:SOT-223-3_TabPin2 -> Package_SO:SOIC-8_3.9x4.9mm_P1.27mm
- moved J1 111.3 mm to (155.9, 48.5), turned to 0 degrees
- moved U1 102.3 mm to (155.6, 56.0), turned to 180 degrees
- moved U2 90.2 mm to (152.9, 71.3), turned to 180 degrees
- moved U3 69.1 mm to (153.8, 64.8), turned to 180 degrees
- moved J2 37.2 mm to (123.7, 52.3), turned to -90 degrees
Connections:
- J1 pad 1: unconnected-(J1-Pad1) -> GND
- J1 pad 10: unconnected-(J1-Pad10) -> /Sensor/sense8
- J1 pad 11: unconnected-(J1-Pad11) -> /Sensor/sense7
- J1 pad 12: unconnected-(J1-Pad12) -> /Sensor/sense6
- J1 pad 13: unconnected-(J1-Pad13) -> /Sensor/sense5
- J1 pad 14: unconnected-(J1-Pad14) -> /Sensor/sense4
- J1 pad 15: unconnected-(J1-Pad15) -> /Sensor/sense3
- J1 pad 16: unconnected-(J1-Pad16) -> /Sensor/sense2
- J1 pad 17: unconnected-(J1-Pad17) -> /Sensor/sense1
- J1 pad 18: unconnected-(J1-Pad18) -> +3V3
- J1 pad 2: unconnected-(J1-Pad2) -> /Sensor/sense16
- J1 pad 3: unconnected-(J1-Pad3) -> /Sensor/sense15
- J1 pad 4: unconnected-(J1-Pad4) -> /Sensor/sense14
- J1 pad 5: unconnected-(J1-Pad5) -> /Sensor/sense13
- J1 pad 6: unconnected-(J1-Pad6) -> /Sensor/sense12
- J1 pad 7: unconnected-(J1-Pad7) -> /Sensor/sense11
- J1 pad 8: unconnected-(J1-Pad8) -> /Sensor/sense10
- J1 pad 9: unconnected-(J1-Pad9) -> /Sensor/sense9
- J2 pad 1: unconnected-(J2-Pin_1-Pad1) -> Net-(J2-Pin_1)
- J2 pad 2: unconnected-(J2-Pin_2-Pad2) -> GND
- U1 pad 1: unconnected-(U1-COMMON_I/O-Pad1) -> /Sensor/Mux_Out
- U1 pad 10: unconnected-(U1-S0-Pad10) -> /MCU/S2
- U1 pad 13: unconnected-(U1-S3-Pad13) -> /MCU/S3
- U1 pad 14: unconnected-(U1-S2-Pad14) -> /MCU/S0
- U1 pad 15: unconnected-(U1-~{E}-Pad15) -> GND
- U1 pad 16: unconnected-(U1-I15-Pad16) -> /Sensor/sense16
- U1 pad 17: unconnected-(U1-I14-Pad17) -> /Sensor/sense15
- U1 pad 18: unconnected-(U1-I13-Pad18) -> /Sensor/sense14
- U1 pad 19: unconnected-(U1-I12-Pad19) -> /Sensor/sense13
- U1 pad 2: unconnected-(U1-I7-Pad2) -> /Sensor/sense1
- U1 pad 20: unconnected-(U1-I11-Pad20) -> /Sensor/sense12
- U1 pad 21: unconnected-(U1-I10-Pad21) -> /Sensor/sense11
- U1 pad 22: unconnected-(U1-I9-Pad22) -> /Sensor/sense10
- U1 pad 23: unconnected-(U1-I8-Pad23) -> /Sensor/sense9
- U1 pad 3: unconnected-(U1-I6-Pad3) -> /Sensor/sense2
- U1 pad 4: unconnected-(U1-I5-Pad4) -> /Sensor/sense3
- U1 pad 5: unconnected-(U1-I4-Pad5) -> /Sensor/sense4
- U1 pad 6: unconnected-(U1-I3-Pad6) -> /Sensor/sense5
- U1 pad 7: unconnected-(U1-I2-Pad7) -> /Sensor/sense6
- U1 pad 8: unconnected-(U1-I1-Pad8) -> /Sensor/sense7
- U1 pad 9: unconnected-(U1-I0-Pad9) -> /Sensor/sense8
- U2 pad 1: unconnected-(U2-VA-Pad1) -> +3V3
- U2 pad 2: unconnected-(U2-GND-Pad2) -> GND
- U2 pad 3: unconnected-(U2-VIN-Pad3) -> Net-(U2-VIN)
- U2 pad 4: unconnected-(U2-SCLK-Pad4) -> /MCU/ADC_CS
- U2 pad 5: unconnected-(U2-SDATA-Pad5) -> /MCU/ADC_SDATA
- U2 pad 6: unconnected-(U2-~{CS}-Pad6) -> /MCU/ADC_CLK
- U3 pad 1: unconnected-(U3-GND-Pad1) -> Net-(U3A--)
- U3 pad 2: unconnected-(U3-VO-Pad2) -> Net-(U3A--)
- U3 pad 3: unconnected-(U3-VI-Pad3) -> /Sensor/Mux_Out
Other:
- board outline added: 44.2 x 48.3 mm

Commit message: idk pcb n shi
Parts:
- removed C1: 0.1u, Capacitor_SMD:C_0603_1608Metric_Pad1.08x0.95mm_HandSolder
- removed C2, C3: 100n, Capacitor_SMD:C_0603_1608Metric_Pad1.08x0.95mm_HandSolder
- removed C7: 10n, Capacitor_SMD:C_0603_1608Metric_Pad1.08x0.95mm_HandSolder
- removed TP1: TestPoint, TestPoint:TestPoint_THTPad_1.0x1.0mm_Drill0.5mm
- added +3v3: TestPoint, TestPoint:TestPoint_THTPad_1.0x1.0mm_Drill0.5mm, F.Cu at (102.6, 104.1)
- added +5V: TestPoint, TestPoint:TestPoint_THTPad_1.0x1.0mm_Drill0.5mm, F.Cu at (108.2, 104.1)
- added C13: 10u, Capacitor_SMD:C_0603_1608Metric_Pad1.08x0.95mm_HandSolder, B.Cu at (84.4, 88.2)
- added C14: 0.1u, Capacitor_SMD:C_0603_1608Metric_Pad1.08x0.95mm_HandSolder, B.Cu at (81.8, 91.3)
- added C15: 1u, Capacitor_SMD:C_0603_1608Metric_Pad1.08x0.95mm_HandSolder, B.Cu at (81.8, 89.5)
- added C16: 10u, Capacitor_SMD:C_0603_1608Metric_Pad1.08x0.95mm_HandSolder, B.Cu at (88.9, 69.0)
- added C17: 1u, Capacitor_SMD:C_0603_1608Metric_Pad1.08x0.95mm_HandSolder, B.Cu at (88.8, 73.6)
- added D1: LED, LED_SMD:LED_0805_2012Metric_Pad1.15x1.40mm_HandSolder, F.Cu at (120.8, 87.2)
- added D2: LED, LED_SMD:LED_1206_3216Metric_Pad1.42x1.75mm_HandSolder, F.Cu at (124.1, 86.9)
- added GND: TestPoint, TestPoint:TestPoint_THTPad_1.0x1.0mm_Drill0.5mm, F.Cu at (105.4, 104.1)
- added J4: Conn_01x04, Connector_PinHeader_2.54mm:PinHeader_1x04_P2.54mm_Vertical, F.Cu at (124.7, 69.0)
- added R11: 10k, Resistor_SMD:R_0603_1608Metric_Pad0.98x0.95mm_HandSolder, F.Cu at (79.7, 77.3)
- added R12: 3k, Resistor_SMD:R_0603_1608Metric_Pad0.98x0.95mm_HandSolder, F.Cu at (124.1, 82.2)
- added SW1: SW_Push, Button_Switch_THT:SW_PUSH_6mm_H5mm, F.Cu at (78.7, 68.7)
- C6: value 10u -> 4.7u; moved to B.Cu
- C8, R7: moved to B.Cu
- R10: value 10k -> 3k
- R8: value 2.2k -> 3k; moved to F.Cu
- R9: value 4k -> 4.4k
- moved J1 91.0 mm to (79.6, 98.0), turned to 90 degrees
- moved U1 80.1 mm to (86.9, 97.2), turned to 0 degrees
- moved R5 80.1 mm to (91.5, 104.3)
- moved R6 71.2 mm to (95.8, 96.5)
- moved R1 71.0 mm to (80.0, 83.6), turned to -90 degrees
- moved C5 69.8 mm to (95.7, 94.9)
- moved U4 67.1 mm to (81.7, 88.0), turned to 0 degrees
- moved U3 66.4 mm to (97.6, 100.2), turned to 0 degrees
- moved R2 63.4 mm to (81.7, 84.5), turned to -90 degrees
- moved C8 60.6 mm to (88.8, 72.1), turned to 0 degrees
- moved C4 60.3 mm to (103.6, 99.2), turned to -90 degrees
- moved U2 54.7 mm to (102.9, 93.5), turned to 0 degrees
- moved J2 46.9 mm to (124.9, 99.1), turned to 0 degrees
- moved R3 44.1 mm to (113.9, 101.4), turned to 90 degrees
- moved C6 43.5 mm to (120.4, 94.0), turned to 180 degrees
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Connections:
- R10 pad 2: Net-(U5-~{CHG}) -> Net-(D1-K)
- U1 pad 11: unconnected-(U1-S1-Pad11) -> /MCU/S1
- U5 pad 14: Net-(U5-TMR) -> unconnected-(U5-TMR-Pad14)
- U5 pad 5: +3V3 -> GND
- U5 pad 9: Net-(U5-~{CHG}) -> Net-(D1-A)
- U6 pad 3: +3V3 -> Net-(U6-EN)
- U6 pad 36: unconnected-(U6-RXD0-Pad36) -> /MCU/Rx_D
- U6 pad 37: unconnected-(U6-TXD0-Pad37) -> /MCU/Tx_D
Routing:
- net /MCU/S1: track 0.00 -> 50.2 mm, vias 0 -> 2
- net /MCU/USB_D_N: track 0.00 -> 40.3 mm, vias 0 -> 2
- net GND: track 0.00 -> 38.0 mm, vias 0 -> 18
- net /MCU/S2: track 0.00 -> 36.8 mm, vias 0 -> 4
- net /MCU/USB_D_P: track 0.00 -> 36.8 mm, vias 0 -> 2
- net /MCU/S3: track 0.00 -> 35.3 mm, vias 0 -> 4
- net /MCU/S0: track 0.00 -> 34.2 mm, vias 0 -> 4
- net /MCU/VDD5V: track 0.00 -> 33.7 mm, vias 0 -> 2
- net /Sensor/Mux_Out: track 0.00 -> 24.8 mm, vias 0 -> 4
- net /MCU/IMU_INT: track 0.00 -> 24.6 mm, vias 0 -> 2
- net /Sensor/sense16: track 0.00 -> 20.3 mm
- net /Sensor/sense15: track 0.00 -> 20.1 mm
- net +3V3: track 0.00 -> 19.5 mm, vias 0 -> 7
- net /MCU/Tx_D: track 0.00 -> 19.1 mm
- net /MCU/Rx_D: track 0.00 -> 18.3 mm, vias 0 -> 1
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- added copper zone on F.Cu, net +3V3
- added copper zone on F.Cu, net /MCU/VDD5V
- added copper zone on B.Cu, net GND
- added copper zone on F.Cu, net Net-(J2-Pin_1)
Other:
- board size 44.2 x 48.3 mm -> 51.4 x 45.9 mm
- board text added: "Impact Insoles V1 ECE445 Spring 26 Group 68"
