File: ImpactInsole_v1/ImpactInsole_v1.kicad_pcb (KiCad board)
At the start: 2 copper layers, 51.4 x 45.9 mm, 40 parts, among them J1 503480-1800, J2 Conn_01x02, J3 USB_C_Receptacle_USB2.0_16P, J4 Conn_01x04, SW1 SW_Push, U1 CD74HC4067SM96, U2 ADC081S021CIMF, U3 OPA1662D, U4 LSM6DSOXTR, U5 BQ24075RGTR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

Commit message: fixed silkscreen warnings
Parts:
- moved R10 0.66 mm to (119.8, 82.8)
Routing:
- net Net-(D1-K): track 2.77 -> 3.43 mm
Other:
- board size 51.4 x 45.9 mm -> 51.7 x 45.9 mm
Changed lines of the file:
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@@
 			(outputformat 1)
 			(mirror no)
-			(drillshape 1)
+			(drillshape 0)
 			(scaleselection 1)
-			(outputdirectory "")
+			(outputdirectory "team68_round1_v1board/")
 		)
 	)
@@
 		(tags "test point THT pad rectangle square")
 		(property "Reference" "+5V"
-			(at -0.07 -1.5 0)
+			(at -0.07 -1.728 0)
 			(layer "F.SilkS")
 			(effects
 				(font
-					(size 0.5 0.5)
+					(size 0.8048 0.5)
 					(thickness 0.125)
 				)
@@
 		(tags "test point THT pad rectangle square")
 		(property "Reference" "GND"
-			(at 0 -1.448 0)
+			(at 0 -1.728 0)
 			(layer "F.SilkS")
 			(effects
 				(font
-					(size 0.5 0.5)
+					(size 0.8048 0.5)
 					(thickness 0.125)
 				)
@@
 		(at 124.88 99.1275)
 		(property "Reference" "J2"
-			(at -1.776 -2.6398 0)
+			(at -2.96 -2.2265 0)
 			(layer "F.SilkS")
 			(effects
 				(font
-					(size 0.48 0.48)
-					(thickness 0.15)
+					(size 0.8102 0.6578)
+					(thickness 0.13156)
+					(bold yes)
 				)
 			)
@@
 	(footprint "Resistor_SMD:R_0603_1608Metric_Pad0.98x0.95mm_HandSolder"
 		(layer "F.Cu")
-		(at 119.78 83.46)
+		(at 119.761 82.804)
 		(descr "Resistor SMD 0603 (1608 Metric), square (rectangular) end terminal, IPC-7351 nominal with elongated pad for handsoldering. (Body size source: IPC-SM-782 page 72, https://www.pcb-3d.com/wordpress/wp-content/uploads/ipc-sm-782a_amendment_1_and_2.pdf), generated with kicad-footprint-generator")
 		(tags "resistor handsolder")
@@
 		(tags "resistor handsolder")
 		(property "Reference" "R6"
-			(at 0 -1.43 0)
+			(at 2.5405 -1.581 0)
 			(layer "F.SilkS")
 			(effects
@@
 		(tags "SOT TO_SOT_SMD")
 		(property "Reference" "U7"
-			(at 0 -2.4 0)
+			(at 1.94 -1.321 0)
 			(layer "F.SilkS")
 			(effects
@@
 		(tags "test point THT pad rectangle square")
 		(property "Reference" "+3v3"
-			(at -0.08 -1.44 0)
+			(at -0.151 -1.728 0)
 			(layer "F.SilkS")
 			(effects
 				(font
-					(size 0.5 0.5)
+					(size 0.8048 0.5)
 					(thickness 0.125)
 				)
@@
 		(at 122.65 92.21 180)
 		(property "Reference" "U5"
-			(at -3.18 2.78 0)
+			(at -3.715 2.167 0)
 			(layer "F.SilkS")
 			(effects
@@
 		(tags "resistor handsolder")
 		(property "Reference" "R9"
-			(at 2.33 0.01 0)
+			(at 2.635 0.012 0)
 			(layer "F.SilkS")
 			(effects
 				(font
-					(size 0.6 0.6)
-					(thickness 0.15)
+					(size 0.9906 0.7874)
+					(thickness 0.12954)
 				)
 			)
@@
 		(tags "SOIC SO")
 		(property "Reference" "U3"
-			(at 0 -3.4 0)
+			(at 0.962 -3.64 0)
 			(layer "F.SilkS")
 			(effects
@@
 		(tags "capacitor handsolder")
 		(property "Reference" "C8"
-			(at 0 1.43 180)
+			(at 2.7495 0.056 180)
 			(layer "B.SilkS")
 			(effects
@@
 	)
 	(gr_rect
-		(start 76.91 59.78)
+		(start 76.529 59.78)
 		(end 128.27 105.68)
 		(stroke
@@
 	)
 	(segment
+		(start 120.6735 83.441)
+		(end 120.6735 82.804)
+		(width 0.2)
+		(layer "F.Cu")
+		(net 38)
+	)
+	(segment
 		(start 120.79 83.5575)
-		(end 120.6925 83.46)
+		(end 120.6735 83.441)
 		(width 0.2)
 		(layer "F.Cu")
