File: ImpactInsole_v1/mcu.kicad_sch (KiCad schematic)
At the start: 9 parts, among them J2 Conn_01x02, J3 USB_C_Receptacle_USB2.0_16P, U5 MCP73831T-2ACI_OT, U6 ESP32-S3-WROOM-1, U7 MCP1700x-300xxTT

Commit message: pcb begnnings + more libs
Parts:
- removed D?: D, symbol Device:D
- removed Q?: PMOS, symbol Simulation_SPICE:PMOS
- removed U5: MCP73831T-2ACI_OT, BMS_Senior_Design:SOT95P280X145-5N, symbol BMS_Senior_Design:MCP73831T-2ACI_OT
- added C10: 1u, Capacitor_SMD:C_0603_1608Metric_Pad1.08x0.95mm_HandSolder, symbol Device:C
- added C6, C9: 10u, Capacitor_SMD:C_0603_1608Metric_Pad1.08x0.95mm_HandSolder, symbol Device:C
- added C7: 10n, Capacitor_SMD:C_0603_1608Metric_Pad1.08x0.95mm_HandSolder, symbol Device:C
- added C8: 0.1u, Capacitor_SMD:C_0603_1608Metric_Pad1.08x0.95mm_HandSolder, symbol Device:C
- added R10, R7: 10k, Resistor_SMD:R_0603_1608Metric_Pad0.98x0.95mm_HandSolder, symbol Device:R
- added R8: 2.2k, Resistor_SMD:R_0603_1608Metric_Pad0.98x0.95mm_HandSolder, symbol Device:R
- added R9: 4k, Resistor_SMD:R_0603_1608Metric_Pad0.98x0.95mm_HandSolder, symbol Device:R
- added TP1: TestPoint, TestPoint:TestPoint_THTPad_1.0x1.0mm_Drill0.5mm, symbol Connector:TestPoint
- added U5: BQ24075RGTR, pp_senior_design:QFN50P300X300X100-17N, symbol PP_Senior_Design:BQ24075RGTR
- J2: footprint (none) -> conn_sen:JST_S2B-PH-K-S_LF__SN_
- R3, R4: footprint Resistor_SMD:R_0805_2012Metric -> Resistor_SMD:R_0603_1608Metric_Pad0.98x0.95mm_HandSolder
Connections:
- net GND: now also J2.2 (Pin_2), U6.1 (GND), U6.40 (GND), U6.41 (GND), U7.1 (GND), C10.2, C6.2, C7.2, C8.2, C9.2, R7.1, R8.1, R9.1, U5.15 (SYSOFF), U5.17 (EXP), U5.4 (~{CE}), U5.8 (VSS)
- net USB_D_N: now also U6.13 (USB_D-)
- net USB_D_P: now also U6.14 (USB_D+)
- net VDD5V: now also C6.1, R10.1, U5.13 (IN)
- net IMU_Data: now reaches U6.12 (IO8)
- net IMU_Clk: now reaches U6.17 (IO9)
- net ADC_CS: now reaches U6.18 (IO10)
- net +3V3: now reaches U6.2 (3V3)
- net +3V3: now also U6.3 (EN), U7.2 (VO), C10.1, C8.1, U5.5 (EN2), U5.6 (EN1)
- net ADC_CLK: now reaches U6.20 (IO12)
- net ADC_SDATA: now reaches U6.21 (IO13)
- net S0: now reaches U6.4 (IO4)
- net S1: now reaches U6.5 (IO5)
- net S2: now reaches U6.6 (IO6)
- net IMU_INT: now reaches U6.7 (IO7)
- net S3: now reaches U6.8 (IO15)
- net at U7.3 (VI): now also C9.1, U5.10 (OUT_10), U5.11 (OUT_11)
- net at J2.1 (Pin_1): now also U5.2 (BAT_2), U5.3 (BAT_3)
- new net: C7.1, U5.14 (TMR)
- new net: R7.2, U5.1 (TS)
- new net: R8.2, U5.12 (ILIM)
- new net: R9.2, U5.16 (ISET)
- new net: TP1.1, U5.7 (~{PGOOD})
- new net: R10.2, U5.9 (~{CHG})
- no-connect marks 3 -> 27
Other:
- moved on the sheet: J2, U7

Commit message: idk pcb n shi
Parts:
- removed C7: 10n, Capacitor_SMD:C_0603_1608Metric_Pad1.08x0.95mm_HandSolder, symbol Device:C
- added C16: 10u, Capacitor_SMD:C_0603_1608Metric_Pad1.08x0.95mm_HandSolder, symbol Device:C
- added C17: 1u, Capacitor_SMD:C_0603_1608Metric_Pad1.08x0.95mm_HandSolder, symbol Device:C
- added D1: LED, LED_SMD:LED_0805_2012Metric_Pad1.15x1.40mm_HandSolder, symbol Device:LED
- added D2: LED, LED_SMD:LED_1206_3216Metric_Pad1.42x1.75mm_HandSolder, symbol Device:LED
- added J4: Conn_01x04, Connector_PinHeader_2.54mm:PinHeader_1x04_P2.54mm_Vertical, symbol Connector_Generic:Conn_01x04
- added R11: 10k, Resistor_SMD:R_0603_1608Metric_Pad0.98x0.95mm_HandSolder, symbol Device:R
- added R12: 3k, Resistor_SMD:R_0603_1608Metric_Pad0.98x0.95mm_HandSolder, symbol Device:R
- added SW1: SW_Push, Button_Switch_THT:SW_PUSH_6mm_H5mm, symbol Switch:SW_Push
- added TP2, TP3: TestPoint, TestPoint:TestPoint_THTPad_1.0x1.0mm_Drill0.5mm, symbol Connector:TestPoint
- C6: value 10u -> 4.7u
- R10: value 10k -> 3k
- R8: value 2.2k -> 3k
- R9: value 4k -> 4.4k
Connections:
- net +3V3: now also TP1.1, C16.1, C17.1, J4.4 (Pin_4), R11.1; no longer U5.5 (EN2), U6.3 (EN)
- net GND: now also U5.5 (EN2), C16.2, C17.2, J4.1 (Pin_1), SW1.1, TP3.1
- net VDD5V: now also R12.2, TP2.1
- net at U5.7 (~{PGOOD}): now also D2.2 (A); no longer TP1.1
- net at U5.9 (~{CHG}): now also D1.2 (A); no longer R10.2
- net Rx_D: now reaches U6.36 (RXD0)
- net Rx_D: now also J4.2 (Pin_2)
- net Tx_D: now reaches U6.37 (TXD0)
- net Tx_D: now also J4.3 (Pin_3)
- new net: D2.1 (K), R12.1
- new net: R11.2, SW1.2, U6.3 (EN)
- new net: D1.1 (K), R10.2
- no-connect marks 27 -> 26
Other:
- moved on the sheet: C6, R10
