File: Flex PCB/Flex PCB.kicad_sch (KiCad schematic)
At the start: 5 parts, among them J1 FPC_Male, J2 Test_Headers

Commit message: Flex PCB v2
Parts:
- added R4, R5, R6, R7: FSR1, Resistor_SMD:FSR_402, symbol Device:R_Variable
- J1: footprint Connector_FFC-FPC:FPC-Male-18P-0.5mm -> Connector_FFC-FPC:FPC-Male-18P-1mm
Connections:
- net 3V3: now also J1.1 (Pin_1), J2.1 (Pin_1), R4.1, R5.1, R6.1, R7.1; no longer J1.18 (Pin_18), J2.18 (Pin_18)
- net at J1.17 (Pin_17), J2.17 (Pin_17): now also R6.2; no longer R1.2
- net at J1.15 (Pin_15), J2.15 (Pin_15): now also R1.2
- net at J1.16 (Pin_16), J2.16 (Pin_16): now also R5.2
- net at J1.2 (Pin_2), J2.2 (Pin_2): now also R7.2; no longer R3.2
- net at J1.3 (Pin_3), J2.3 (Pin_3): now also R4.2
- net at J1.4 (Pin_4), J2.4 (Pin_4): now also R3.2
- new net GND: J1.18 (Pin_18), J2.18 (Pin_18)
