File: Flex Hub PCB/Flex Hub PCB.kicad_pcb (KiCad board)
At the start: 2 copper layers, 58.5 x 98 mm, 3 parts, among them J1 Conn_01x18_Socket, J2 Conn_01x18_Socket, J3 Conn_01x18_Socket

Commit message: Final flex designs and gerbers
Other:
- outline, holes or cut-outs redrawn
- board text added: "ImpactInsoles FlexHubV1 ECE445 Spring 26 Group 68"
Changed lines of the file:
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@@
 			(outputformat 1)
 			(mirror no)
-			(drillshape 1)
+			(drillshape 0)
 			(scaleselection 1)
-			(outputdirectory "")
+			(outputdirectory "Gerbers/")
 		)
 	)
@@
 	(gr_line
 		(start 131 32.5)
-		(end 90 32.5)
+		(end 92 32.5)
 		(stroke
 			(width 0.05)
@@
 		(layer "Edge.Cuts")
 	)
+	(gr_arc
+		(start 92 55)
+		(mid 90.585786 54.414214)
+		(end 90 53)
+		(stroke
+			(width 0.05)
+			(type default)
+		)
+		(layer "Edge.Cuts")
+	)
 	(gr_line
 		(start 122 60)
@@
 	)
 	(gr_line
-		(start 90 32.5)
-		(end 90 55)
+		(start 90 34.5)
+		(end 90 53)
 		(stroke
 			(width 0.05)
@@
 	)
 	(gr_line
-		(start 90 55)
+		(start 92 55)
 		(end 113 55)
 		(stroke
@@
 		(layer "Edge.Cuts")
 	)
+	(gr_arc
+		(start 90 34.5)
+		(mid 90.585786 33.085786)
+		(end 92 32.5)
+		(stroke
+			(width 0.05)
+			(type default)
+		)
+		(layer "Edge.Cuts")
+	)
+	(gr_text "ImpactInsoles\nFlexHubV1\nECE445 Spring 26\nGroup 68\n"
+		(at 129 56.5 0)
+		(layer "F.SilkS")
+		(effects
+			(font
+				(size 0.8984 0.8984)
+				(thickness 0.14986)
+				(bold yes)
+			)
+			(justify left bottom)
+		)
+	)
 	(segment
