File: Right Angle Extension/RAFlexExt/RAFlexExt.kicad_pcb (KiCad board)
At the start: 2 copper layers, 29 x 51.8 mm, 2 parts, among them J1 Conn_01x18_Pin, J2 Conn_01x18_Socket

Commit message: After all r4 edits (late)
Other:
- board text added: "Stiffener TOP"
Changed lines of the file:
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@@
 		(35 "F.Fab" user)
 		(33 "B.Fab" user)
-		(39 "User.1" user)
+		(39 "User.1" user "F.Stiffener_PI_0.2mm")
 		(41 "User.2" user)
 		(43 "User.3" user)
@@
 		(tenting front back)
 		(pcbplotparams
-			(layerselection 0x00000000_00000000_55555555_5755f5ff)
+			(layerselection 0x00000000_00000000_555555d5_575df5ff)
 			(plot_on_all_layers_selection 0x00000000_00000000_00000000_00000000)
 			(disableapertmacros no)
-			(usegerberextensions no)
+			(usegerberextensions yes)
 			(usegerberattributes yes)
 			(usegerberadvancedattributes yes)
-			(creategerberjobfile yes)
+			(creategerberjobfile no)
 			(dashed_line_dash_ratio 12.000000)
 			(dashed_line_gap_ratio 3.000000)
@@
 			(drillshape 0)
 			(scaleselection 1)
-			(outputdirectory "Gerbers/")
+			(outputdirectory "Gerbers_Stiffener/")
 		)
 	)
@@
 		)
 	)
+	(gr_text "Stiffener TOP"
+		(at 158.1 77.7 0)
+		(layer "Cmts.User")
+		(effects
+			(font
+				(size 1 1)
+				(thickness 0.15)
+			)
+			(justify left bottom)
+		)
+	)
 	(dimension
 		(type orthogonal)
 		(layer "Cmts.User")
 		(pts
-			(xy 160 75.5921) (xy 162 130.5921)
-		)
-		(height 9)
+			(xy 148.2 75.3) (xy 148.2 78.8)
+		)
+		(height 8.7)
 		(orientation 1)
 		(format
@@
 		)
 		(style
-			(thickness 0.2)
+			(thickness 0.1)
 			(arrow_length 1.27)
 			(text_position_mode 0)
@@
 			(keep_text_aligned yes)
 		)
-		(gr_text "55"
-			(at 167.2 103.0921 90)
+		(gr_text "3.5"
+			(at 155.75 77.05 90)
 			(layer "Cmts.User")
 			(effects
 				(font
-					(size 1.5 1.5)
-					(thickness 0.3)
+					(size 1 1)
+					(thickness 0.15)
 				)
 			)
