File: Short Flex/Flex PCB.kicad_pcb (KiCad board)
At the start: 2 copper layers, 74.8 x 68.5 mm, 9 parts, among them J1 FPC_Male, J2 Test_Headers

Commit message: Final flex designs and gerbers
Other:
- board text added: "ImpactInsoles ShortFlex ECE445 Spring 26 Group 68"
- board text removed: "ImpactInsoles Flex V2 ECE445 Spring 26 Group 68"
Changed lines of the file:
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@@
 		(layer "Edge.Cuts")
 	)
-	(gr_text "ImpactInsoles\nFlex V2\nECE445 Spring 26\nGroup 68\n"
+	(gr_text "ImpactInsoles\nShortFlex\nECE445 Spring 26\nGroup 68\n"
 		(at 179.5 99.725 90)
 		(layer "F.SilkS")
